File: nixiedice.sch (KiCad schematic (older format))
At the start: 47 parts, among them CON1 BARREL_JACK, P1 USB_OTG, P2 USB_A, P3 ARDUINO PRO MICRO, P8 CONN_01X04, Q1 MPSA42, Q2 MPSA42, Q3 MPSA42, SW1 SW_PUSH, SW2 SW_PUSH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

Commit message: change microusb connector to use smd pads
also add line on front silkscreen to plug this schweet repo
Connections:
- no-connect marks 17 -> 18
Changed lines of the file:
@@
 Text Notes 800  7600 0    60   ~ 0
 Maybe you'll want to do something with these? idk
+NoConn ~ 2650 4350
 $EndSCHEMATC
