File: nixiedice.kicad_pcb (KiCad board)
At the start: 2 copper layers, 127 x 63.5 mm, 51 parts, among them CON1 BARREL_JACK, M1 1pin, M2 1pin, M3 1pin, M4 1pin, P1 USB_OTG, P2 USB_A, P3 ARDUINO PRO MICRO, P8 CONN_01X04, Q1 MPSA42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

Commit message: emergency pcb silkscreen revision
Other:
- board text added: "Rev Bee"
- board text removed: "Rev B"
Changed lines of the file:
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@@
-(kicad_pcb (version 4) (host pcbnew 4.0.4-stable)
+(kicad_pcb (version 4) (host pcbnew 4.0.5)
   (general
     (links 170)
@@
     (effects (font (size 1.27 1.143) (thickness 0.254)))
   )
-  (gr_text "Rev B" (at 43.434 3.048) (layer F.SilkS)
+  (gr_text "Rev Bee" (at 44.7 3.048) (layer F.SilkS)
     (effects (font (size 1.5 1.5) (thickness 0.3)))
   )
